Commit message: Add Gazebo simulation for mobile robot

File: src/mobile_robot_description/urdf/common_properties.xacro (robot description, xacro)
@@ -1,4 +1,9 @@
 <?xml version="1.0"?>
 <robot xmlns:xacro="https://www.ros.org/wiki/xacro">
+    <xacro:property name="base_length" value="0.8" />
+    <xacro:property name="base_width" value="0.5" />
+    <xacro:property name="base_height" value="0.2" />
+    <xacro:property name="wheel_radius" value="0.1" />
+    <xacro:property name="wheel_length" value="0.05" />
     <material name="green">
         <color rgba="0 0.6 0 1" />
@@ -7,3 +12,30 @@
         <color rgba="0.7 0.7 0.7 1" />
     </material>
+    <xacro:macro name="box_inertia" params="m x y z o_xyz o_rpy">
+        <inertial>
+            <mass value="${m}" />
+            <origin xyz="${o_xyz}" rpy="${o_rpy}" />
+            <inertia ixx="${(m / 12) * (z * z + y * y)}" ixy="0" ixz="0"
+                     iyy="${(m / 12) * (x * x + z * z)}" iyz="0"
+                     izz="${(m / 12) * (x * x + y * y)}" />
+        </inertial>
+    </xacro:macro>
+    <xacro:macro name="cylinder_inertia" params="m r l o_xyz o_rpy">
+        <inertial>
+            <mass value="${m}" />
+            <origin xyz="${o_xyz}" rpy="${o_rpy}" />
+            <inertia ixx="${(m / 12) * (3 * r * r + l * l)}" ixy="0" ixz="0"
+                     iyy="${(m / 12) * (3 * r * r + l * l)}" iyz="0"
+                     izz="${(m / 2) * (r * r)}" />
+        </inertial>
+    </xacro:macro>
+    <xacro:macro name="sphere_inertia" params="m r o_xyz o_rpy">
+        <inertial>
+            <mass value="${m}" />
+            <origin xyz="${o_xyz}" rpy="${o_rpy}" />
+            <inertia ixx="${(2 / 5) * m * r * r}" ixy="0" ixz="0"
+                     iyy="${(2 / 5) * m * r * r}" iyz="0"
+                     izz="${(2 / 5) * m * r * r}" />
+        </inertial>
+    </xacro:macro>
 </robot>

File: src/mobile_robot_description/urdf/mobile_base.xacro (robot description, xacro)
@@ -1,9 +1,4 @@
 <?xml version="1.0"?>
 <robot xmlns:xacro="https://www.ros.org/wiki/xacro">
-    <xacro:property name="base_length" value="0.8" />
-    <xacro:property name="base_width" value="0.5" />
-    <xacro:property name="base_height" value="0.2" />
-    <xacro:property name="wheel_radius" value="0.1" />
-    <xacro:property name="wheel_length" value="0.05" />
     <link name="base_footprint" />
     <link name="base_link">
@@ -15,4 +10,12 @@
             <material name="green" />
         </visual>
+        <collision>
+            <geometry>
+                <box size="${base_length} ${base_width} ${base_height}" />
+            </geometry>
+            <origin xyz="0 0 ${base_height / 2.0}" rpy="0 0 0" />
+        </collision>
+        <xacro:box_inertia m="6.0" x="${base_length}" y="${base_width}" z="${base_height}"
+                           o_xyz="0 0 ${base_height / 2.0}" o_rpy="0 0 0" />
     </link>
     <xacro:macro name="wheel_link" params="prefix">
@@ -26,10 +29,18 @@
                 <material name="gray" />
             </visual>
+            <collision>
+                <geometry>
+                    <sphere radius="${wheel_radius}" />
+                </geometry>
+                <origin xyz="0 0 0" rpy="0 0 0" />
+            </collision>
+            <xacro:cylinder_inertia m="1.0" r="${wheel_radius}" l="${wheel_length}"
+                                    o_xyz="0 0 0" o_rpy="${pi / 2.0} 0 0" />
         </link>
     </xacro:macro>
     <xacro:wheel_link prefix="front_right" />
     <xacro:wheel_link prefix="front_left" />
-    <xacro:wheel_link prefix="back_right" />
-    <xacro:wheel_link prefix="back_left" />
+    <xacro:wheel_link prefix="rear_right" />
+    <xacro:wheel_link prefix="rear_left" />
     <joint name="base_joint" type="fixed">
         <parent link="base_footprint" />
@@ -49,13 +60,13 @@
         <axis xyz="0 1 0" />
     </joint>
-    <joint name="base_back_right_wheel_joint" type="continuous">
+    <joint name="base_rear_right_wheel_joint" type="continuous">
         <parent link="base_link" />
-        <child link="back_right_wheel_link" />
+        <child link="rear_right_wheel_link" />
         <origin xyz="${-base_length / 4.0} ${-(base_width + wheel_length) / 2.0} 0" rpy="0 0 0" />
         <axis xyz="0 1 0" />
     </joint>
-    <joint name="base_back_left_wheel_joint" type="continuous">
+    <joint name="base_rear_left_wheel_joint" type="continuous">
         <parent link="base_link" />
-        <child link="back_left_wheel_link" />
+        <child link="rear_left_wheel_link" />
         <origin xyz="${-base_length / 4.0} ${(base_width + wheel_length) / 2.0} 0" rpy="0 0 0" />
         <axis xyz="0 1 0" />

File: src/mobile_robot_description/urdf/mobile_robot.urdf.xacro (robot description, xacro)
@@ -3,3 +3,4 @@
     <xacro:include filename="$(find mobile_robot_description)/urdf/common_properties.xacro" />
     <xacro:include filename="$(find mobile_robot_description)/urdf/mobile_base.xacro" />
+    <xacro:include filename="$(find mobile_robot_description)/urdf/mobile_base_gazebo.xacro" />
 </robot>
